File: PCB Files/trigger_switch_pcb.sch (EAGLE design)
At the start: 7 parts

Commit message: update to wiring diagram
i think i have the board schematic done!   All grounds on the bottom,
all signals on the top
Connections:
- net GND: now also U$1.GND
Changed lines of the file:
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@@
 <label x="-5.08" y="58.42" size="1.778" layer="95"/>
+</segment>
+<segment>
+<pinref part="U$1" gate="G$1" pin="GND"/>
+<wire x1="22.86" y1="83.82" x2="17.78" y2="83.82" width="0.1524" layer="91"/>
+<label x="15.24" y="83.82" size="1.778" layer="95"/>
 </segment>
 </net>
